Commit message: STarted simplification

File: MATLAB/Collision_test.urdf (robot description, URDF)
Before this commit: robot Collision_Test, 24 links, 23 joints
Links:
- link 70I_v1_1: geometry collision mesh filename=C:\Users\atjensvo\cernbox\Documents\GitHub\MasterThesis\MAT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 scale=0.001 0.001 0.001; visual mesh filename=C:\Users\atjensvo\cernbox\Documents\GitHub\MasterThesis\MAT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 scale=0.001 0.001 0.001
- link 70I_v3_1: geometry collision mesh filename=C:\Users\atjensvo\cernbox\Documents\GitHub\MasterThesis\MAT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 scale=0.001 0.001 0.001; visual mesh filename=C:\Users\atjensvo\cernbox\Documents\GitHub\MasterThesis\MAT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 scale=0.001 0.001 0.001
- link 70mm_Connector_v8_1: geometry collision mesh filename=C:\Users\atjensvo\cernbox\Documents\GitHub\MasterThesis\MAT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 scale=0.001 0.001 0.001; visual mesh filename=C:\Users\atjensvo\cernbox\Documents\GitHub\MasterThesis\MAT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 scale=0.001 0.001 0.001
- link 70mm_Connector_v8__1__1: geometry collision mesh filename=C:\Users\atjensvo\cernbox\Documents\GitHub\MasterThesis\MAT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 scale=0.001 0.001 0.001; visual mesh filename=C:\Users\atjensvo\cernbox\Documents\GitHub\MasterThesis\MAT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 scale=0.001 0.001 0.001
- link 70mm_Short_v1_1: geometry collision mesh filename=C:\Users\atjensvo\cernbox\Documents\GitHub\MasterThesis\MAT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 scale=0.001 0.001 0.001; visual mesh filename=C:\Users\atjensvo\cernbox\Documents\GitHub\MasterThesis\MAT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 scale=0.001 0.001 0.001
- link 70mm_Short_v1__1__1: geometry collision mesh filename=C:\Users\atjensvo\cernbox\Documents\GitHub\MasterThesis\MAT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 scale=0.001 0.001 0.001; visual mesh filename=C:\Users\atjensvo\cernbox\Documents\GitHub\MasterThesis\MAT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 scale=0.001 0.001 0.001
- link 80I_v1_1: geometry collision mesh filename=C:\Users\atjensvo\cernbox\Documents\GitHub\MasterThesis\MAT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 scale=0.001 0.001 0.001; visual mesh filename=C:\Users\atjensvo\cernbox\Documents\GitHub\MasterThesis\MAT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 scale=0.001 0.001 0.001
- link 80I_v2_1: geometry collision mesh filename=C:\Users\atjensvo\cernbox\Documents\GitHub\MasterThesis\MAT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 scale=0.001 0.001 0.001; visual mesh filename=C:\Users\atjensvo\cernbox\Documents\GitHub\MasterThesis\MAT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 scale=0.001 0.001 0.001
- link 80I_v7_1: geometry collision mesh filename=C:\Users\atjensvo\cernbox\Documents\GitHub\MasterThesis\MAT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 scale=0.001 0.001 0.001; visual mesh filename=C:\Users\atjensvo\cernbox\Documents\GitHub\MasterThesis\MAT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 scale=0.001 0.001 0.001
- link 80mm_Connector_v1_1: geometry collision mesh filename=C:\Users\atjensvo\cernbox\Documents\GitHub\MasterThesis\MAT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 scale=0.001 0.001 0.001; visual mesh filename=C:\Users\atjensvo\cernbox\Documents\GitHub\MasterThesis\MAT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 scale=0.001 0.001 0.001
- link 80mm_Connector_v1_2: geometry collision mesh filename=C:\Users\atjensvo\cernbox\Documents\GitHub\MasterThesis\MAT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 scale=0.001 0.001 0.001; visual mesh filename=C:\Users\atjensvo\cernbox\Documents\GitHub\MasterThesis\MAT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 scale=0.001 0.001 0.001
- link J0_roll_v2_1: geometry collision mesh filename=C:\Users\atjensvo\cernbox\Documents\GitHub\MasterThesis\MAT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 scale=0.001 0.001 0.001; visual mesh filename=C:\Users\atjensvo\cernbox\Documents\GitHub\MasterThesis\MAT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 scale=0.001 0.001 0.001
- link J1_pitch_v1_1: geometry collision mesh filename=C:\Users\atjensvo\cernbox\Documents\GitHub\MasterThesis\MAT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 scale=0.001 0.001 0.001; visual mesh filename=C:\Users\atjensvo\cernbox\Documents\GitHub\MasterThesis\MAT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 scale=0.001 0.001 0.001
- link J2_prismatic_v2_1: geometry collision mesh filename=C:\Users\atjensvo\cernbox\Documents\GitHub\MasterThesis\MAT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 scale=0.001 0.001 0.001; visual mesh filename=C:\Users\atjensvo\cernbox\Documents\GitHub\MasterThesis\MAT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 scale=0.001 0.001 0.001
- link Ph11_v5_1: geometry collision mesh filename=C:\Users\atjensvo\cernbox\Documents\GitHub\MasterThesis\MAT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 scale=0.001 0.001 0.001; visual mesh filename=C:\Users\atjensvo\cernbox\Documents\GitHub\MasterThesis\MAT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 scale=0.001 0.001 0.001
- link Ph14_v3_1: geometry collision mesh filename=C:\Users\atjensvo\cernbox\Documents\GitHub\MasterThesis\MAT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 scale=0.001 0.001 0.001; visual mesh filename=C:\Users\atjensvo\cernbox\Documents\GitHub\MasterThesis\MAT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 scale=0.001 0.001 0.001
- link Ph14_v3__1__1: geometry collision mesh filename=C:\Users\atjensvo\cernbox\Documents\GitHub\MasterThesis\MAT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 scale=0.001 0.001 0.001; visual mesh filename=C:\Users\atjensvo\cernbox\Documents\GitHub\MasterThesis\MAT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 scale=0.001 0.001 0.001
- link Ph17_v3_1: geometry collision mesh filename=C:\Users\atjensvo\cernbox\Documents\GitHub\MasterThesis\MAT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 scale=0.001 0.001 0.001; visual mesh filename=C:\Users\atjensvo\cernbox\Documents\GitHub\MasterThesis\MAT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 scale=0.001 0.001 0.001
- link Ph17_v5_1: geometry collision mesh filename=C:\Users\atjensvo\cernbox\Documents\GitHub\MasterThesis\MAT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 scale=0.001 0.001 0.001; visual mesh filename=C:\Users\atjensvo\cernbox\Documents\GitHub\MasterThesis\MAT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 scale=0.001 0.001 0.001
- link Ph_14_v5_1: geometry collision mesh filename=C:\Users\atjensvo\cernbox\Documents\GitHub\MasterThesis\MAT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 scale=0.001 0.001 0.001; visual mesh filename=C:\Users\atjensvo\cernbox\Documents\GitHub\MasterThesis\MAT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 scale=0.001 0.001 0.001
- link Ph_14_v5__1__1: geometry collision mesh filename=C:\Users\atjensvo\cernbox\Documents\GitHub\MasterThesis\MAT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 scale=0.001 0.001 0.001; visual mesh filename=C:\Users\atjensvo\cernbox\Documents\GitHub\MasterThesis\MAT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 scale=0.001 0.001 0.001
- link Tool_1: geometry collision mesh filename=C:\Users\atjensvo\cernbox\Documents\GitHub\MasterThesis\MAT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 scale=0.001 0.001 0.001; visual mesh filename=C:\Users\atjensvo\cernbox\Documents\GitHub\MasterThesis\MAT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 scale=0.001 0.001 0.001
- link Wagon_slider_1: geometry collision mesh filename=C:\Users\atjensvo\cernbox\Documents\GitHub\MasterThesis\MAT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 scale=0.001 0.001 0.001; visual mesh filename=C:\Users\atjensvo\cernbox\Documents\GitHub\MasterThesis\MAT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 scale=0.001 0.001 0.001
- link base_link: geometry collision mesh filename=C:\Users\atjensvo\cernbox\Documents\GitHub\MasterThesis\MAT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 scale=0.001 0.001 0.001; visual mesh filename=C:\Users\atjensvo\cernbox\Documents\GitHub\MasterThesis\MAT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 scale=0.001 0.001 0.001
